File: self-balan.sch (EAGLE design)
At the start: 15 parts, among them U1 ATMEGA328P_TQFP

Commit message: Minor fix
Parts:
- added C8: (no value), rcl:C-USC0805
- added JP1: (no value), pinhead:PINHD-2X3
- added Q1: (no value), adafruit:CRYSTALHC18U-V
- added S1: (no value), switch-omron:10-XX
- added UART-HEADER: (no value), pinhead:PINHD-1X4
Connections:
- new net +5V: R3.2
- new net GND: C2.1, C2.2, C8.2, JP1.6, Q1.2, S1.P, S1.P1, U1.PB6(XTAL1/TOSC1), UART-HEADER.4
- new net MISO: JP1.1, U1.PB4(MISO)
- new net MOSI: JP1.4, U1.PB3(MOSI/OC2)
- new net N$3: C3.2, U1.AGND, U1.GND@3, U1.GND@5
- new net N$4: C8.1, Q1.1, U1.PB7(XTAL2/TOSC2)
- new net RST: JP1.5, R3.1, S1.S, S1.S1, U1.PC6(/RESET)
- new net RXD: U1.PD1(TXD), UART-HEADER.2
- new net SCK: JP1.3, U1.PB5(SCK)
- new net TXD: U1.PD0(RXD), UART-HEADER.1
- new net VCC: C3.1, JP1.2, U1.AREF, U1.AVCC, U1.VCC@4, U1.VCC@6, UART-HEADER.3
Other:
- moved on the sheet: C2, C3, R1, R2, R3

Commit message: minor fixes
Parts:
- removed C1, C4, C5, C7: (no value), rcl:C-USC0805
- removed R1, R2, R4, R5, R6, R7: (no value), rcl:R-US_R0805
- added C9: 10u, rcl:C-USC0805
- added IC1: 7805T, linear:7805T
- added U$1, U$2: A4988_STEP, IC:A4988_STEP
- added X1: (no value), con-wago-508:W237-02P
- C6: value (none) -> 10u
Connections:
- net +5V: now also C3.1, C9.1, IC1.VO, JP1.2, U1.AREF, U1.AVCC, U1.VCC@4, U1.VCC@6, UART-HEADER.3
- net GND: now also C6.2, C9.2, IC1.GND, X1-2.KL
- net VCC: now also C6.1, IC1.VI, X1-1.KL; no longer C3.1, JP1.2, U1.AREF, U1.AVCC, U1.VCC@4, U1.VCC@6, UART-HEADER.3
Other:
- moved on the sheet: C2, C3, C6, C8, JP1, Q1, R3, S1, U1, UART-HEADER

Commit message: Routing fixes
Parts:
- added C1, C4: 100u, rcl:C-USC0805
- added U$3, U$4: JST-PH_4-PIN_HEADER, SRG:JST-PH_4-PIN_HEADER
- added U2: GY-521MPU6050, gy-521:GY-521MPU6050
- renumbered U$1 to RIGHT, U$2 to LEFT
Connections:
- new net D10: U1.PB2(SS/OC1B)
- new net D3: U1.PD3(INT1)
- new net D4: LEFT./EN, RIGHT./EN, U1.PD4(XCK/T0)
- new net D5: RIGHT.STEP, U1.PD5(T1)
- new net D6: LEFT.STEP, U1.PD6(AIN0)
- new net D7: RIGHT.DIR, U1.PD7(AIN1)
- new net D8: LEFT.DIR, U1.PB0(ICP)
- new net D9: U1.PB1(OC1A)
- new net INT: U1.PD2(INT0), U2.INT
- new net N$10: RIGHT.1A, U$3.1
- new net N$11: LEFT.2B, U$4.4
- new net N$12: LEFT.2A, U$4.3
- new net N$13: RIGHT./RST, RIGHT./SLP
- new net N$14: LEFT.1B, U$4.2
- new net N$15: LEFT.1A, U$4.1
- new net N$16: LEFT./RST, LEFT./SLP
- new net N$7: RIGHT.2B, U$3.4
- new net N$8: RIGHT.2A, U$3.3
- new net N$9: RIGHT.1B, U$3.2
- new net SCL: U1.PC5(ADC5/SCL), U2.SCL
- new net SDA: U1.PC4(ADC4/SDA), U2.SDA
- net +5V: now also LEFT.MS1, LEFT.MS2, LEFT.VDD, RIGHT.MS1, RIGHT.MS2, RIGHT.VDD, U2.VCC, UART-HEADER.4; no longer UART-HEADER.3
- net GND: now also C1.2, C4.2, LEFT.GND, LEFT.MS3, RIGHT.GND, RIGHT.MS3, U2.GND, UART-HEADER.3; no longer UART-HEADER.4
- net VCC: now also C1.1, C4.1, LEFT.VMOT, RIGHT.VMOT
